Commit message: sync latest parameters

File: replace_ros_odrive/odrive_botwheel_explorer/description/urdf/diffbot_description.urdf.xacro (robot description, xacro)
@@ -163,5 +163,5 @@
         <parent link="base_link"/>
         <child link="camera_link"/>
-        <origin xyz="${realsense_xoff} ${realsense_yoff} ${(base_height/2-realsense_zoff)}" rpy="0 0 0"/>
+        <origin xyz="${realsense_xoff} ${realsense_yoff} ${(base_height/2-realsense_zoff)}" rpy="0 0.05 0"/>
     </joint>
     <!-- Realsense body -->
